File: basketweave_bottom/basketweave_bottom.kicad_pcb (KiCad board)
At the start: 2 copper layers, 371.5 x 145.3 mm, 16 parts

Commit message: changed logo, name, and pattern design
Parts:
- removed the G*** at (200.0, 155.6)
- removed H10, H12: MountingHole, MountingHole:MountingHole_2.2mm_M2_Pad
- added G***: LOGO, basketweave_bottom:logo_bottom, B.Cu at (205.6, 140.5)
- moved H9 27.8 mm to (378.6, 181.0)
- moved H8 3.97 mm to (38.9, 181.8)
Routing:
- added copper zone on F.Cu, net (none)
Other:
- board text removed: "Designed by Noah L"
- board text removed: "clackery.com"
