File: basketweave/basketweave.kicad_pcb (KiCad board)
At the start: 2 copper layers, 371.5 x 145.3 mm, 176 parts, among them SW3 Rotary_Encoder_Switch, U1 ATmega32A-PU, Y1 16Mhz

Commit message: changed logo, name, and pattern design
Parts:
- removed the G*** at (215.9, 206.4)
- removed H10, H12: MountingHole, MountingHole:MountingHole_2.2mm_M2_Pad
- removed MX72: MX-NoLED, MX_Only:MXOnly-3U-ReversedStabilizers-NoLED
- removed MX73: MX-NoLED, MX_Only:MXOnly-1.25U-NoLED
- added D72: D_Small, Diode_THT:D_DO-35_SOD27_P7.62mm_Horizontal, F.Cu at (375.5, 119.1)
- added G***: LOGO, basketweave:logo, B.Cu at (89.7, 196.1)
- added MX70: MX-NoLED, MX_Only:MXOnly-2.25U-ReversedStabilizers-NoLED, F.Cu at (152.8, 203.6)
- added MX71: MX-NoLED, MX_Only:MXOnly-1U-NoLED, F.Cu at (183.1, 210.1)
- added REF**: pattern_right, basketweave:pattern_right, F.Cu at (254.0, 86.5)
- added REF**: pattern_left, basketweave:pattern_left, F.Cu at (40.5, 86.5)
- ROTARY ENCODER: renamed from SW3
- moved H9 27.8 mm to (381.0, 188.1)
- moved H8 3.97 mm to (41.3, 188.9)
Connections:
- net RGBIN renamed Net-(U1-Pad4)
- ROTARY ENCODER pad S2: ROW4 -> Net-(D72-Pad2)
- USB pad S1: (no net) -> GND
Routing:
- net ROW4: track 464.5 -> 453.7 mm
- net Net-(D72-Pad2): track 0.00 -> 7.47 mm
- net COL8: track 110.6 -> 108.1 mm
- net COL10: track 141.0 -> 138.5 mm
- net Net-(D62-Pad2): track 222.2 -> 224.7 mm
- net COL6: track 106.0 -> 108.5 mm
- net COL4: track 160.3 -> 162.7 mm
- net Net-(D61-Pad2): track 197.0 -> 199.4 mm
Other:
- board text added: "Rev 1"
- board text added: "github.com/null-ll/basketweave"
- board text removed: "JLCJLCJLCJLC"

Commit message: added switch size markings
Other:
- board text added: "1.25u"
- board text added: "1u"
- board text added: "2.25u"
- board text added: "2u"
- board text added: "Normal"
- board text added: "Stepped"
